Commit message: imported patch urdf

File: models/myravenII_source.urdf (robot description, URDF)
Before this commit: robot raven_2, 42 links, 41 joints
Joints:
- joint elbow_L: limit lower=-3.1415 upper=3.1415 effort=1000.0 velocity=0.5 -> lower=0.785398163 upper=2.35619449 effort=1000.0 velocity=0.5
- joint elbow_R: limit lower=-3.1415 upper=3.1415 effort=1000.0 velocity=0.5 -> lower=0.785398163 upper=2.35619449 effort=1000.0 velocity=0.5
- joint grasper_joint_1_L: limit lower=-2 upper=2 effort=1000.0 velocity=.5 -> lower=-1.55334303 upper=1.55334303 effort=1000.0 velocity=.5
- joint grasper_joint_1_R: limit lower=-2 upper=2 effort=1000.0 velocity=.5 -> lower=-1.55334303 upper=1.55334303 effort=1000.0 velocity=.5
- joint grasper_joint_2_L: limit lower=-2 upper=2 effort=1000.0 velocity=.5 -> lower=-1.55334303 upper=1.55334303 effort=1000.0 velocity=.5
- joint grasper_joint_2_R: limit lower=-2 upper=2 effort=1000.0 velocity=.5 -> lower=-1.55334303 upper=1.55334303 effort=1000.0 velocity=.5
- joint grasper_yaw_L: limit lower=-2 upper=2 effort=1000.0 velocity=.5 -> lower=-1.57079633 upper=1.57079633 effort=1000.0 velocity=.5
- joint grasper_yaw_R: limit lower=-2 upper=2 effort=1000.0 velocity=.5 -> lower=-1.57079633 upper=1.57079633 effort=1000.0 velocity=.5
- joint insertion_L: limit lower=-.17 upper=.1 effort=1000.0 velocity=0.5 -> lower=-.230 upper=.010 effort=1000.0 velocity=0.5
- joint insertion_R: limit lower=-.17 upper=.1 effort=1000.0 velocity=0.5 -> lower=-.230 upper=.010 effort=1000.0 velocity=0.5
- joint shoulder_L: limit lower=-3.1415 upper=3.1415 effort=1000.0 velocity=0.5 -> lower=0.0 upper=1.57079633 effort=1000.0 velocity=0.5
- joint shoulder_R: limit lower=-3.1415 upper=3.1415 effort=1000.0 velocity=0.5 -> lower=0.0 upper=1.57079633 effort=1000.0 velocity=0.5
- joint tool_roll_L: limit lower=-3.1415 upper=3.1415 effort=1000.0 velocity=0.5 -> lower=-3.17649924 upper=3.17649924 effort=1000.0 velocity=0.5
- joint tool_roll_R: limit lower=-3.1415 upper=3.1415 effort=1000.0 velocity=0.5 -> lower=-3.17649924 upper=3.17649924 effort=1000.0 velocity=0.5
- joint wrist_joint_L: limit lower=-2 upper=2 effort=1000.0 velocity=0.5 -> lower=-1.30899694 upper=1.30899694 effort=1000.0 velocity=0.5
- joint wrist_joint_R: limit lower=-2 upper=2 effort=1000.0 velocity=0.5 -> lower=-1.30899694 upper=1.30899694 effort=1000.0 velocity=0.5

Commit message: Update raven collada file to new base_mount_R value

File: models/myravenII_source.urdf (robot description, URDF)
Before this commit: robot raven_2, 42 links, 41 joints
Joints:
- joint base_mount_R: origin xyz=-0.14858 0.002 0 rpy=0 0 1.5707963267948966 -> xyz=-0.149 0.005 -0.006 rpy=0 0 1.5707963267948966
